File: kicad/DigitalControl.sch (KiCad schematic (older format))
At the start: 9 parts, among them U1 ILQ74

Commit message: Adding untracked files
Connections:
- net CS: now also R2.2; no longer R3.2
- net CS_ISOLATED: now also R6.1, U1.14; no longer R7.1, U1.11
- net MUTE: now also R1.2; no longer R4.2
- net MUTE_ISOLATED: now also R5.1, U1.15; no longer R8.1, U1.10
- net SCL: now also R4.2; no longer R1.2
- net SCL_ISOLATED: now also R8.1, U1.10; no longer R5.1, U1.15
- net SDA: now also R3.2; no longer R2.2
- net SDA_ISOLATED: now also R7.1, U1.11; no longer R6.1, U1.14
Changed lines of the file:
@@
 	1    0    0    -1
 $EndComp
+Text HLabel 3450 4550 0    60   Input ~ 0
+SCL
+Text HLabel 3450 3950 0    60   Input ~ 0
+SDA
+Text HLabel 3450 3350 0    60   Input ~ 0
+CS
 Text HLabel 3450 2750 0    60   Input ~ 0
-SCL
-Text HLabel 3450 3350 0    60   Input ~ 0
-SDA
-Text HLabel 3450 3950 0    60   Input ~ 0
-CS
-Text HLabel 3450 4550 0    60   Input ~ 0
 MUTE
 Text HLabel 3450 5150 0    60   Input ~ 0
@@
 $EndComp
 $Comp
-L +5VD #PWR09
+L +5VD #PWR011
 U 1 1 56CAE58F
 P 7150 2400
-F 0 "#PWR09" H 7150 2250 50  0001 C CNN
+F 0 "#PWR011" H 7150 2250 50  0001 C CNN
 F 1 "+5VD" H 7150 2540 50  0000 C CNN
 F 2 "" H 7150 2400 50  0000 C CNN
@@
 	5950 2950 5950 5150
 $Comp
-L GNDD #PWR010
+L GNDD #PWR012
 U 1 1 56CAEA1B
 P 5950 5150
-F 0 "#PWR010" H 5950 4900 50  0001 C CNN
+F 0 "#PWR012" H 5950 4900 50  0001 C CNN
 F 1 "GNDD" H 5950 5000 50  0000 C CNN
 F 2 "" H 5950 5150 50  0000 C CNN
@@
 	5650 4750 5950 4750
 Connection ~ 5950 4750
+Text HLabel 7600 4550 2    60   Input ~ 0
+SCL_ISOLATED
+Text HLabel 7600 3950 2    60   Input ~ 0
+SDA_ISOLATED
+Text HLabel 7600 3350 2    60   Input ~ 0
+CS_ISOLATED
 Text HLabel 7600 2750 2    60   Input ~ 0
-SCL_ISOLATED
-Text HLabel 7600 3350 2    60   Input ~ 0
-SDA_ISOLATED
-Text HLabel 7600 3950 2    60   Input ~ 0
-CS_ISOLATED
-Text HLabel 7600 4550 2    60   Input ~ 0
 MUTE_ISOLATED
 $EndSCHEMATC
