File: kicad/Digital_Control.sch (KiCad schematic (older format))
At the start: 14 parts, among them IC1 ATMEGA328P-P, P9 ICSP, SW1 SPST, Y1 16MHz

Commit message: Produced Volume knob including Gerbers, and updated main board to remove ERC errors.  Just about to start board layout
Parts:
- removed SW1: SPST, symbol SPST
- added C13: 0.1u, Capacitors_SMD:C_0603_HandSoldering, symbol C
- added D2: 0, LEDs:LED_1206, symbol Led_Small
- added R13: 220, Resistors_SMD:R_0603_HandSoldering, symbol R
- added R18: 10k, Resistors_SMD:R_0603_HandSoldering, symbol R
- added SW1: SW_PUSH, Buttons_Switches_SMD:SW_SPST_B3S-1000, symbol SW_PUSH
- C14: renamed from C10; footprint (none) -> Capacitors_SMD:C_0603_HandSoldering
- C15: renamed from C11; footprint (none) -> Capacitors_SMD:C_0603_HandSoldering
- D3: renamed from D2; footprint (none) -> LEDs:LED_1206
- D4: renamed from D3; footprint (none) -> LEDs:LED_1206
- D5: renamed from D4; footprint (none) -> LEDs:LED_1206
- D6: renamed from D5; footprint (none) -> LEDs:LED_1206
- IC1: footprint DIL28 -> Housings_DIP:DIP-28_W7.62mm
- P10: renamed from P9; footprint (none) -> Pin_Headers:Pin_Header_Straight_2x03
- R14: renamed from R9; footprint (none) -> Resistors_SMD:R_0603_HandSoldering
- R15: renamed from R10; footprint (none) -> Resistors_SMD:R_0603_HandSoldering
- R16: renamed from R11; footprint (none) -> Resistors_SMD:R_0603_HandSoldering
- R17: renamed from R12; footprint (none) -> Resistors_SMD:R_0603_HandSoldering
- Y1: footprint (none) -> Crystals:Crystal_HC49-U_Vertical
Connections:
- net labels added: PA_ENABLE, SCLK, SDI
- net labels removed: SCL, SDA
- wire segments 29 -> 39
Changed lines of the file:
@@
 Text HLabel 1650 4800 0    60   Input ~ 0
 CS
-Text HLabel 1650 5000 0    60   Input ~ 0
-SDA
-Text HLabel 1650 5200 0    60   Input ~ 0
-SCL
 $Comp
 L ATMEGA328P-P IC1
@@
 F 0 "IC1" H 4500 4800 50  0000 L BNN
 F 1 "ATMEGA328P-P" H 5650 2150 50  0000 L BNN
-F 2 "DIL28" H 5250 3550 50  0000 C CIN
+F 2 "Housings_DIP:DIP-28_W7.62mm" H 5250 3550 50  0000 C CIN
 F 3 "" H 5250 3550 50  0000 C CNN
 	1    5250 3550
@@
 Text Label 1650 2200 0    60   ~ 0
 RX_IN
-Text Label 6250 3700 0    60   ~ 0
-SDA
-Text Label 6250 3800 0    60   ~ 0
-SCL
-Text Label 1650 5000 0    60   ~ 0
-SDA
-Text Label 1650 5200 0    60   ~ 0
-SCL
 Text Label 6250 2550 0    60   ~ 0
 ROT_A
@@
 CS
 $Comp
-L GNDD #PWR30
+L GNDD #PWR046
 U 1 1 575F1469
 P 4200 4900
-F 0 "#PWR30" H 4200 4650 50  0001 C CNN
+F 0 "#PWR046" H 4200 4650 50  0001 C CNN
 F 1 "GNDD" H 4200 4750 50  0000 C CNN
 F 2 "" H 4200 4900 50  0000 C CNN
@@
 $EndComp
 $Comp
-L +5VD #PWR29
+L +5VD #PWR047
 U 1 1 575F147F
 P 4200 2300
-F 0 "#PWR29" H 4200 2150 50  0001 C CNN
+F 0 "#PWR047" H 4200 2150 50  0001 C CNN
 F 1 "+5VD" H 4200 2440 50  0000 C CNN
 F 2 "" H 4200 2300 50  0000 C CNN
@@
 	4350 2450 4200 2450
 Wire Wire Line
-	4200 2300 4200 3050
+	4200 2300 4200 3500
 Wire Wire Line
 	4200 2750 4350 2750
@@
 Connection ~ 4200 2750
 Wire Wire Line
-	4350 4750 4200 4750
-Wire Wire Line
-	4200 4650 4200 4900
+	4200 4750 4350 4750
+Wire Wire Line
+	4200 3800 4200 4900
 Wire Wire Line
 	4350 4650 4200 4650
 Connection ~ 4200 4750
 $Comp
-L CONN_02X03 P9
+L CONN_02X03 P10
 U 1 1 575FD1F4
 P 9700 1300
-F 0 "P9" H 9700 1500 50  0000 C CNN
+F 0 "P10" H 9700 1500 50  0000 C CNN
 F 1 "ICSP" H 9700 1100 50  0000 C CNN
-F 2 "" H 9700 100 50  0000 C CNN
+F 2 "Pin_Headers:Pin_Header_Straight_2x03" H 9700 100 50  0001 C CNN
 F 3 "" H 9700 100 50  0000 C CNN
 	1    9700 1300
@@
 MOSI
 $Comp
-L +5VD #PWR33
+L +5VD #PWR048
 U 1 1 575FD2AB
 P 9950 1200
-F 0 "#PWR33" H 9950 1050 50  0001 C CNN
+F 0 "#PWR048" H 9950 1050 50  0001 C CNN
 F 1 "+5VD" H 9950 1340 50  0000 C CNN
 F 2 "" H 9950 1200 50  0000 C CNN
@@
 $EndComp
 $Comp
-L GNDD #PWR34
+L GNDD #PWR049
 U 1 1 575FD2C3
 P 9950 1400
-F 0 "#PWR34" H 9950 1150 50  0001 C CNN
+F 0 "#PWR049" H 9950 1150 50  0001 C CNN
 F 1 "GNDD" H 9950 1250 50  0000 C CNN
 F 2 "" H 9950 1400 50  0000 C CNN
@@
 	8000 3500 8000 3800
 $Comp
-L Led_Small D2
+L Led_Small D3
 U 1 1 575FD761
 P 7700 3900
-F 0 "D2" H 7650 4025 50  0000 L CNN
+F 0 "D3" H 7650 4025 50  0000 L CNN
 F 1 "1" H 7700 3800 50  0000 L CNN
-F 2 "" V 7700 3900 50  0000 C CNN
+F 2 "LEDs:LED_1206" V 7700 3900 50  0001 C CNN
 F 3 "" V 7700 3900 50  0000 C CNN
 	1    7700 3900
@@
 $EndComp
 $Comp
-L Led_Small D3
+L Led_Small D4
 U 1 1 575FD78F
 P 8000 3900
-F 0 "D3" H 7950 4025 50  0000 L CNN
+F 0 "D4" H 7950 4025 50  0000 L CNN
 F 1 "2" H 8000 3800 50  0000 L CNN
-F 2 "" V 8000 3900 50  0000 C CNN
+F 2 "LEDs:LED_1206" V 8000 3900 50  0001 C CNN
 F 3 "" V 8000 3900 50  0000 C CNN
 	1    8000 3900
@@
 $EndComp
 $Comp
-L R R9
+L R R14
 U 1 1 575FD80A
 P 7700 4150
-F 0 "R9" V 7780 4150 50  0000 C CNN
+F 0 "R14" V 7780 4150 50  0000 C CNN
 F 1 "220" V 7700 4150 50  0000 C CNN
-F 2 "" V 7630 4150 50  0000 C CNN
+F 2 "Resistors_SMD:R_0603_HandSoldering" V 7630 4150 50  0001 C CNN
 F 3 "" H 7700 4150 50  0000 C CNN
 	1    7700 4150
@@
 $EndComp
 $Comp
-L R R10
+L R R15
 U 1 1 575FD830
 P 8000 4150
-F 0 "R10" V 8080 4150 50  0000 C CNN
+F 0 "R15" V 8080 4150 50  0000 C CNN
 F 1 "220" V 8000 4150 50  0000 C CNN
-F 2 "" V 7930 4150 50  0000 C CNN
+F 2 "Resistors_SMD:R_0603_HandSoldering" V 7930 4150 50  0001 C CNN
 F 3 "" H 8000 4150 50  0000 C CNN
 	1    8000 4150
@@
 $EndComp
 $Comp
-L SPST SW1
-U 1 1 575FD8F8
-P 9200 4500
-F 0 "SW1" H 9200 4600 50  0000 C CNN
-F 1 "SPST" H 9200 4400 50  0000 C CNN
-F 2 "" H 9200 4500 50  0000 C CNN
-F 3 "" H 9200 4500 50  0000 C CNN
-	1    9200 4500
-	1    0    0    -1
-$EndComp
-$Comp
-L GNDD #PWR32
+L GNDD #PWR050
 U 1 1 575FD92F
-P 9700 4500
-F 0 "#PWR32" H 9700 4250 50  0001 C CNN
-F 1 "GNDD" H 9700 4350 50  0000 C CNN
-F 2 "" H 9700 4500 50  0000 C CNN
-F 3 "" H 9700 4500 50  0000 C CNN
-	1    9700 4500
+P 8700 4500
+F 0 "#PWR050" H 8700 4250 50  0001 C CNN
+F 1 "GNDD" H 8700 4350 50  0000 C CNN
+F 2 "" H 8700 4500 50  0000 C CNN
+F 3 "" H 8700 4500 50  0000 C CNN
+	1    8700 4500
 	1    0    0    -1
 $EndComp
@@
 	7700 4300 7700 4500
 Wire Wire Line
-	7700 4500 8700 4500
+	7400 4500 8700 4500
 Wire Wire Line
 	8000 4300 8000 4500
@@
 SOURCE_2_ENABLE
 $Comp
-L Led_Small D4
+L Led_Small D5
 U 1 1 57600105
 P 8300 3900
-F 0 "D4" H 8250 4025 50  0000 L CNN
+F 0 "D5" H 8250 4025 50  0000 L CNN
 F 1 "S1" H 8300 3800 50  0000 L CNN
-F 2 "" V 8300 3900 50  0000 C CNN
+F 2 "LEDs:LED_1206" V 8300 3900 50  0001 C CNN
 F 3 "" V 8300 3900 50  0000 C CNN
 	1    8300 3900
@@
 $EndComp
 $Comp
-L Led_Small D5
+L Led_Small D6
 U 1 1 5760010B
 P 8600 3900
-F 0 "D5" H 8550 4025 50  0000 L CNN
+F 0 "D6" H 8550 4025 50  0000 L CNN
 F 1 "S2" H 8600 3800 50  0000 L CNN
-F 2 "" V 8600 3900 50  0000 C CNN
+F 2 "LEDs:LED_1206" V 8600 3900 50  0001 C CNN
 F 3 "" V 8600 3900 50  0000 C CNN
 	1    8600 3900
@@
 $EndComp
 $Comp
-L R R11
+L R R16
 U 1 1 57600111
 P 8300 4150
-F 0 "R11" V 8380 4150 50  0000 C CNN
+F 0 "R16" V 8380 4150 50  0000 C CNN
 F 1 "220" V 8300 4150 50  0000 C CNN
-F 2 "" V 8230 4150 50  0000 C CNN
+F 2 "Resistors_SMD:R_0603_HandSoldering" V 8230 4150 50  0001 C CNN
 F 3 "" H 8300 4150 50  0000 C CNN
 	1    8300 4150
@@
 $EndComp
 $Comp
-L R R12
+L R R17
 U 1 1 57600117
 P 8600 4150
-F 0 "R12" V 8680 4150 50  0000 C CNN
+F 0 "R17" V 8680 4150 50  0000 C CNN
 F 1 "220" V 8600 4150 50  0000 C CNN
-F 2 "" V 8530 4150 50  0000 C CNN
+F 2 "Resistors_SMD:R_0603_HandSoldering" V 8530 4150 50  0001 C CNN
 F 3 "" H 8600 4150 50  0000 C CNN
 	1    8600 4150
 	1    0    0    -1
 $EndComp
-Wire Wire Line
-	8300 4300 8300 4500
-Wire Wire Line
-	8600 4300 8600 4500
 Wire Wire Line
 	6250 3400 8300 3400
@@
 F 0 "Y1" H 7000 3050 50  0000 C CNN
 F 1 "16MHz" H 7000 2850 50  0000 C CNN
-F 2 "" H 7000 2950 50  0000 C CNN
+F 2 "Crystals:Crystal_HC49-U_Vertical" H 7000 2950 50  0001 C CNN
 F 3 "" H 7000 2950 50  0000 C CNN
 	1    7000 2950
@@
 $EndComp
 $Comp
-L C C10
+L C C14
 U 1 1 57604478
 P 7150 2700
-F 0 "C10" H 7175 2800 50  0000 L CNN
+F 0 "C14" H 7175 2800 50  0000 L CNN
 F 1 "22p" H 7175 2600 50  0000 L CNN
-F 2 "" H 7188 2550 50  0000 C CNN
+F 2 "Capacitors_SMD:C_0603_HandSoldering" H 7188 2550 50  0001 C CNN
 F 3 "" H 7150 2700 50  0000 C CNN
 	1    7150 2700
@@
 $EndComp
 $Comp
-L C C11
+L C C15
 U 1 1 576044B9
 P 7150 3150
-F 0 "C11" H 7175 3250 50  0000 L CNN
+F 0 "C15" H 7175 3250 50  0000 L CNN
 F 1 "22p" H 7175 3050 50  0000 L CNN
-F 2 "" H 7188 3000 50  0000 C CNN
+F 2 "Capacitors_SMD:C_0603_HandSoldering" H 7188 3000 50  0001 C CNN
 F 3 "" H 7150 3150 50  0000 C CNN
 	1    7150 3150
@@
 $EndComp
 $Comp
-L GNDD #PWR31
+L GNDD #PWR051
 U 1 1 5760462A
 P 7500 3000
-F 0 "#PWR31" H 7500 2750 50  0001 C CNN
+F 0 "#PWR051" H 7500 2750 50  0001 C CNN
 F 1 "GNDD" H 7500 2850 50  0000 C CNN
 F 2 "" H 7500 3000 50  0000 C CNN
@@
 	7500 2950 7500 3000
 Connection ~ 7300 2950
+Wire Wire Line
+	8300 4300 8300 4500
+Connection ~ 8300 4500
+Wire Wire Line
+	8600 4300 8600 4500
+Connection ~ 8600 4500
+$Comp
+L SW_PUSH SW1
+U 1 1 57611910
+P 8500 1400
+F 0 "SW1" H 8650 1510 50  0000 C CNN
+F 1 "SW_PUSH" H 8500 1320 50  0000 C CNN
+F 2 "Buttons_Switches_SMD:SW_SPST_B3S-1000" H 8500 1400 50  0001 C CNN
+F 3 "" H 8500 1400 50  0000 C CNN
+	1    8500 1400
+	1    0    0    -1
+$EndComp
+$Comp
+L GNDD #PWR052
+U 1 1 57611977
+P 8200 1400
+F 0 "#PWR052" H 8200 1150 50  0001 C CNN
+F 1 "GNDD" H 8200 1250 50  0000 C CNN
+F 2 "" H 8200 1400 50  0000 C CNN
+F 3 "" H 8200 1400 50  0000 C CNN
+	1    8200 1400
+	1    0    0    -1
+$EndComp
+$Comp
+L R R18
+U 1 1 576119B8
+P 8950 1250
+F 0 "R18" V 9030 1250 50  0000 C CNN
+F 1 "10k" V 8950 1250 50  0000 C CNN
+F 2 "Resistors_SMD:R_0603_HandSoldering" V 8880 1250 50  0001 C CNN
+F 3 "" H 8950 1250 50  0000 C CNN
+	1    8950 1250
+	1    0    0    -1
+$EndComp
+$Comp
+L +5VD #PWR053
+U 1 1 57611A51
+P 8950 1100
+F 0 "#PWR053" H 8950 950 50  0001 C CNN
+F 1 "+5VD" H 8950 1240 50  0000 C CNN
+F 2 "" H 8950 1100 50  0000 C CNN
+F 3 "" H 8950 1100 50  0000 C CNN
+	1    8950 1100
+	1    0    0    -1
+$EndComp
+Wire Wire Line
+	8800 1400 9450 1400
+Connection ~ 8950 1400
+$Comp
+L C C13
+U 1 1 57611D76
+P 4200 3650
+F 0 "C13" H 4225 3750 50  0000 L CNN
+F 1 "0.1u" H 4225 3550 50  0000 L CNN
+F 2 "Capacitors_SMD:C_0603_HandSoldering" H 4238 3500 50  0001 C CNN
+F 3 "" H 4200 3650 50  0000 C CNN
+	1    4200 3650
+	1    0    0    -1
+$EndComp
+Connection ~ 4200 3050
+Connection ~ 4200 4650
+Text HLabel 1650 3800 0    60   Input ~ 0
+PA_ENABLE
+Text Label 1650 3800 0    60   ~ 0
+PA_ENABLE
+Text Label 6250 3800 0    60   ~ 0
+PA_ENABLE
+$Comp
+L Led_Small D2
+U 1 1 57612D24
+P 7400 3900
+F 0 "D2" H 7350 4025 50  0000 L CNN
+F 1 "0" H 7400 3800 50  0000 L CNN
+F 2 "LEDs:LED_1206" V 7400 3900 50  0001 C CNN
+F 3 "" V 7400 3900 50  0000 C CNN
+	1    7400 3900
+	0    -1   -1   0
+$EndComp
+$Comp
+L R R13
+U 1 1 57612D2A
+P 7400 4150
+F 0 "R13" V 7480 4150 50  0000 C CNN
+F 1 "220" V 7400 4150 50  0000 C CNN
+F 2 "Resistors_SMD:R_0603_HandSoldering" V 7330 4150 50  0001 C CNN
+F 3 "" H 7400 4150 50  0000 C CNN
+	1    7400 4150
+	1    0    0    -1
+$EndComp
+Wire Wire Line
+	7400 4300 7400 4500
+Wire Wire Line
+	6250 3700 7400 3700
+Wire Wire Line
+	7400 3700 7400 3800
+Connection ~ 7700 4500
+Text HLabel 6500 1600 0    60   Input ~ 0
+SDI
+Text HLabel 6500 1750 0    60   Input ~ 0
+SCLK
+Wire Wire Line
+	6250 2750 6600 2750
+Wire Wire Line
+	6600 2750 6600 1600
+Wire Wire Line
+	6600 1600 6500 1600
+Wire Wire Line
+	6250 2950 6700 2950
+Wire Wire Line
+	6700 2950 6700 1750
+Wire Wire Line
+	6700 1750 6500 1750
 $EndSCHEMATC

Commit message: Routed the board.  Passes ERC check
Parts:
- D5: value S1 -> S2
- D6: value S2 -> S1
Changed lines of the file:
@@
 P 8300 3900
 F 0 "D5" H 8250 4025 50  0000 L CNN
-F 1 "S1" H 8300 3800 50  0000 L CNN
+F 1 "S2" H 8300 3800 50  0000 L CNN
 F 2 "LEDs:LED_1206" V 8300 3900 50  0001 C CNN
 F 3 "" V 8300 3900 50  0000 C CNN
@@
 P 8600 3900
 F 0 "D6" H 8550 4025 50  0000 L CNN
-F 1 "S2" H 8600 3800 50  0000 L CNN
+F 1 "S1" H 8600 3800 50  0000 L CNN
 F 2 "LEDs:LED_1206" V 8600 3900 50  0001 C CNN
 F 3 "" V 8600 3900 50  0000 C CNN

Commit message: Updated to include extra indicator LEDs controlled by the ATMega.  PCB reworked
Parts:
- removed D2: 0, LEDs:LED_1206, symbol Led_Small
- removed R13: 220, Resistors_SMD:R_0603_HandSoldering, symbol R
- added Q4: NXP2301P, TO_SOT_Packages_SMD:SOT-23_Handsoldering, symbol Q_PMOS_GSD
- added R22: 10k, Resistors_SMD:R_0603_HandSoldering, symbol R
- D3, D4, D5, D6: footprint LEDs:LED_1206 -> SMD_LED:LED_SMD_1.6x0.8mm
Connections:
- net GNDD: now also Q4.2 (S), R22.2; no longer R14.2, R15.2, R16.2, R17.2
- net at IC1.27 ((PCINT12/SDA/ADC4)PC4): now also Q4.1 (G), R22.1
- new net LED_GND: Q4.3 (D), R14.2, R15.2, R16.2, R17.2
Changed lines of the file:
@@
 F 0 "D3" H 7650 4025 50  0000 L CNN
 F 1 "1" H 7700 3800 50  0000 L CNN
-F 2 "LEDs:LED_1206" V 7700 3900 50  0001 C CNN
+F 2 "SMD_LED:LED_SMD_1.6x0.8mm" V 7700 3900 50  0001 C CNN
 F 3 "" V 7700 3900 50  0000 C CNN
 	1    7700 3900
@@
 F 0 "D4" H 7950 4025 50  0000 L CNN
 F 1 "2" H 8000 3800 50  0000 L CNN
-F 2 "LEDs:LED_1206" V 8000 3900 50  0001 C CNN
+F 2 "SMD_LED:LED_SMD_1.6x0.8mm" V 8000 3900 50  0001 C CNN
 F 3 "" V 8000 3900 50  0000 C CNN
 	1    8000 3900
@@
 L GNDD #PWR050
 U 1 1 575FD92F
-P 8700 4500
-F 0 "#PWR050" H 8700 4250 50  0001 C CNN
-F 1 "GNDD" H 8700 4350 50  0000 C CNN
-F 2 "" H 8700 4500 50  0000 C CNN
-F 3 "" H 8700 4500 50  0000 C CNN
-	1    8700 4500
+P 7400 5150
+F 0 "#PWR050" H 7400 4900 50  0001 C CNN
+F 1 "GNDD" H 7400 5000 50  0000 C CNN
+F 2 "" H 7400 5150 50  0000 C CNN
+F 3 "" H 7400 5150 50  0000 C CNN
+	1    7400 5150
 	1    0    0    -1
 $EndComp
@@
 F 0 "D5" H 8250 4025 50  0000 L CNN
 F 1 "S2" H 8300 3800 50  0000 L CNN
-F 2 "LEDs:LED_1206" V 8300 3900 50  0001 C CNN
+F 2 "SMD_LED:LED_SMD_1.6x0.8mm" V 8300 3900 50  0001 C CNN
 F 3 "" V 8300 3900 50  0000 C CNN
 	1    8300 3900
@@
 F 0 "D6" H 8550 4025 50  0000 L CNN
 F 1 "S1" H 8600 3800 50  0000 L CNN
-F 2 "LEDs:LED_1206" V 8600 3900 50  0001 C CNN
+F 2 "SMD_LED:LED_SMD_1.6x0.8mm" V 8600 3900 50  0001 C CNN
 F 3 "" V 8600 3900 50  0000 C CNN
 	1    8600 3900
@@
 Text Label 6250 3800 0    60   ~ 0
 PA_ENABLE
-$Comp
-L Led_Small D2
-U 1 1 57612D24
-P 7400 3900
-F 0 "D2" H 7350 4025 50  0000 L CNN
-F 1 "0" H 7400 3800 50  0000 L CNN
-F 2 "LEDs:LED_1206" V 7400 3900 50  0001 C CNN
-F 3 "" V 7400 3900 50  0000 C CNN
-	1    7400 3900
-	0    -1   -1   0
-$EndComp
-$Comp
-L R R13
-U 1 1 57612D2A
-P 7400 4150
-F 0 "R13" V 7480 4150 50  0000 C CNN
-F 1 "220" V 7400 4150 50  0000 C CNN
-F 2 "Resistors_SMD:R_0603_HandSoldering" V 7330 4150 50  0001 C CNN
-F 3 "" H 7400 4150 50  0000 C CNN
-	1    7400 4150
-	1    0    0    -1
-$EndComp
-Wire Wire Line
-	7400 4300 7400 4500
-Wire Wire Line
-	6250 3700 7400 3700
-Wire Wire Line
-	7400 3700 7400 3800
 Connection ~ 7700 4500
 Text HLabel 6500 1600 0    60   Input ~ 0
@@
 Wire Wire Line
 	6700 1750 6500 1750
+$Comp
+L Q_PMOS_GSD Q4
+U 1 1 5762E45C
+P 7300 4700
+F 0 "Q4" H 7600 4750 50  0000 R CNN
+F 1 "NXP2301P" H 7950 4650 50  0000 R CNN
+F 2 "TO_SOT_Packages_SMD:SOT-23_Handsoldering" H 7500 4800 50  0001 C CNN
+F 3 "" H 7300 4700 50  0000 C CNN
+	1    7300 4700
+	1    0    0    -1
+$EndComp
+$Comp
+L R R22
+U 1 1 5762E527
+P 7100 4850
+F 0 "R22" V 7180 4850 50  0000 C CNN
+F 1 "10k" V 7100 4850 50  0000 C CNN
+F 2 "Resistors_SMD:R_0603_HandSoldering" V 7030 4850 50  0001 C CNN
+F 3 "" H 7100 4850 50  0000 C CNN
+	1    7100 4850
+	1    0    0    -1
+$EndComp
+Wire Wire Line
+	7100 5000 7400 5000
+Wire Wire Line
+	7400 4900 7400 5150
+Connection ~ 7400 5000
+Wire Wire Line
+	7100 4700 7100 3700
+Wire Wire Line
+	7100 3700 6250 3700
+Text GLabel 8700 4500 2    60   Input ~ 0
+LED_GND
 $EndSCHEMATC

Commit message: Minor updates and board submitted for fabrication
Parts:
- removed Q4: NXP2301P, TO_SOT_Packages_SMD:SOT-23_Handsoldering, symbol Q_PMOS_GSD
- added D12: RX, SMD_LED:LED_SMD_1.6x0.8mm, symbol Led_Small
- added D13: TX, SMD_LED:LED_SMD_1.6x0.8mm, symbol Led_Small
- added D14: MISO, SMD_LED:LED_SMD_1.6x0.8mm, symbol Led_Small
- added D15: MOSI, SMD_LED:LED_SMD_1.6x0.8mm, symbol Led_Small
- added Q4: TSM2302CX, TO_SOT_Packages_SMD:SOT-23_Handsoldering, symbol Q_NMOS_GSD
- added R25, R26, R27, R28: 220, Resistors_SMD:R_0603_HandSoldering, symbol R
Connections:
- net GNDD: now also Q4.2 (S)
- net LED_GND: now also Q4.3 (D), R25.2, R26.2, R27.2, R28.2
- net MISO: now also D14.2 (A)
- net RX_IN: now also D12.2 (A)
- net SDI: now also D15.2 (A)
- net TX_OUT: now also D13.2 (A)
- net at IC1.27 ((PCINT12/SDA/ADC4)PC4), R22.1: now also Q4.1 (G)
- new net: D13.1 (K), R26.1
- new net: D12.1 (K), R25.1
- new net: D15.1 (K), R28.1
- new net: D14.1 (K), R27.1
Other:
- moved on the sheet: C14, C15, Y1
Changed lines of the file:
@@
 L Crystal_Small Y1
 U 1 1 576043F5
-P 7000 2950
-F 0 "Y1" H 7000 3050 50  0000 C CNN
-F 1 "16MHz" H 7000 2850 50  0000 C CNN
-F 2 "Crystals:Crystal_HC49-U_Vertical" H 7000 2950 50  0001 C CNN
-F 3 "" H 7000 2950 50  0000 C CNN
-	1    7000 2950
+P 9450 2950
+F 0 "Y1" H 9450 3050 50  0000 C CNN
+F 1 "16MHz" H 9450 2850 50  0000 C CNN
+F 2 "Crystals:Crystal_HC49-U_Vertical" H 9450 2950 50  0001 C CNN
+F 3 "" H 9450 2950 50  0000 C CNN
+	1    9450 2950
 	0    1    1    0
 $EndComp
@@
 L C C14
 U 1 1 57604478
-P 7150 2700
-F 0 "C14" H 7175 2800 50  0000 L CNN
-F 1 "22p" H 7175 2600 50  0000 L CNN
-F 2 "Capacitors_SMD:C_0603_HandSoldering" H 7188 2550 50  0001 C CNN
-F 3 "" H 7150 2700 50  0000 C CNN
-	1    7150 2700
+P 9600 2700
+F 0 "C14" H 9625 2800 50  0000 L CNN
+F 1 "22p" H 9625 2600 50  0000 L CNN
+F 2 "Capacitors_SMD:C_0603_HandSoldering" H 9638 2550 50  0001 C CNN
+F 3 "" H 9600 2700 50  0000 C CNN
+	1    9600 2700
 	0    1    1    0
 $EndComp
@@
 L C C15
 U 1 1 576044B9
-P 7150 3150
-F 0 "C15" H 7175 3250 50  0000 L CNN
-F 1 "22p" H 7175 3050 50  0000 L CNN
-F 2 "Capacitors_SMD:C_0603_HandSoldering" H 7188 3000 50  0001 C CNN
-F 3 "" H 7150 3150 50  0000 C CNN
-	1    7150 3150
+P 9600 3150
+F 0 "C15" H 9625 3250 50  0000 L CNN
+F 1 "22p" H 9625 3050 50  0000 L CNN
+F 2 "Capacitors_SMD:C_0603_HandSoldering" H 9638 3000 50  0001 C CNN
+F 3 "" H 9600 3150 50  0000 C CNN
+	1    9600 3150
 	0    1    1    0
 $EndComp
@@
 L GNDD #PWR051
 U 1 1 5760462A
-P 7500 3000
-F 0 "#PWR051" H 7500 2750 50  0001 C CNN
-F 1 "GNDD" H 7500 2850 50  0000 C CNN
-F 2 "" H 7500 3000 50  0000 C CNN
-F 3 "" H 7500 3000 50  0000 C CNN
-	1    7500 3000
-	1    0    0    -1
-$EndComp
-Wire Wire Line
-	6250 3150 7000 3150
-Wire Wire Line
-	7000 3150 7000 3050
-Wire Wire Line
-	7000 2850 7000 2700
-Wire Wire Line
-	7000 2700 6750 2700
-Wire Wire Line
-	6750 2700 6750 3050
-Wire Wire Line
-	6750 3050 6250 3050
-Wire Wire Line
-	7300 2700 7300 3150
-Wire Wire Line
-	7300 2950 7500 2950
-Wire Wire Line
-	7500 2950 7500 3000
-Connection ~ 7300 2950
+P 9950 3000
+F 0 "#PWR051" H 9950 2750 50  0001 C CNN
+F 1 "GNDD" H 9950 2850 50  0000 C CNN
+F 2 "" H 9950 3000 50  0000 C CNN
+F 3 "" H 9950 3000 50  0000 C CNN
+	1    9950 3000
+	1    0    0    -1
+$EndComp
+Wire Wire Line
+	6250 3150 9450 3150
+Wire Wire Line
+	9450 3150 9450 3050
+Wire Wire Line
+	9450 2850 9450 2700
+Wire Wire Line
+	9450 2700 9200 2700
+Wire Wire Line
+	6250 3050 9200 3050
+Wire Wire Line
+	9750 2700 9750 3150
+Wire Wire Line
+	9750 2950 9950 2950
+Wire Wire Line
+	9950 2950 9950 3000
+Connection ~ 9750 2950
 Wire Wire Line
 	8300 4300 8300 4500
@@
 	6600 2750 6600 1600
 Wire Wire Line
-	6600 1600 6500 1600
+	6500 1600 7550 1600
 Wire Wire Line
 	6250 2950 6700 2950
@@
 Wire Wire Line
 	6700 1750 6500 1750
-$Comp
-L Q_PMOS_GSD Q4
-U 1 1 5762E45C
-P 7300 4700
-F 0 "Q4" H 7600 4750 50  0000 R CNN
-F 1 "NXP2301P" H 7950 4650 50  0000 R CNN
-F 2 "TO_SOT_Packages_SMD:SOT-23_Handsoldering" H 7500 4800 50  0001 C CNN
-F 3 "" H 7300 4700 50  0000 C CNN
-	1    7300 4700
-	1    0    0    -1
-$EndComp
 $Comp
 L R R22
@@
 Text GLabel 8700 4500 2    60   Input ~ 0
 LED_GND
+$Comp
+L Q_NMOS_GSD Q4
+U 1 1 5763AB02
+P 7300 4700
+F 0 "Q4" H 7600 4750 50  0000 R CNN
+F 1 "TSM2302CX" H 7950 4650 50  0000 R CNN
+F 2 "TO_SOT_Packages_SMD:SOT-23_Handsoldering" H 7500 4800 50  0001 C CNN
+F 3 "" H 7300 4700 50  0000 C CNN
+	1    7300 4700
+	1    0    0    -1
+$EndComp
+$Comp
+L Led_Small D13
+U 1 1 5763AFC9
+P 3150 2400
+F 0 "D13" H 3100 2525 50  0000 L CNN
+F 1 "TX" H 3150 2300 50  0000 L CNN
+F 2 "SMD_LED:LED_SMD_1.6x0.8mm" V 3150 2400 50  0001 C CNN
+F 3 "" V 3150 2400 50  0000 C CNN
+	1    3150 2400
+	0    -1   -1   0
+$EndComp
+$Comp
+L R R26
+U 1 1 5763AFCF
+P 3150 2650
+F 0 "R26" V 3230 2650 50  0000 C CNN
+F 1 "220" V 3150 2650 50  0000 C CNN
+F 2 "Resistors_SMD:R_0603_HandSoldering" V 3080 2650 50  0001 C CNN
+F 3 "" H 3150 2650 50  0000 C CNN
+	1    3150 2650
+	1    0    0    -1
+$EndComp
+$Comp
+L Led_Small D12
+U 1 1 5763B19A
+P 2800 2400
+F 0 "D12" H 2750 2525 50  0000 L CNN
+F 1 "RX" H 2800 2300 50  0000 L CNN
+F 2 "SMD_LED:LED_SMD_1.6x0.8mm" V 2800 2400 50  0001 C CNN
+F 3 "" V 2800 2400 50  0000 C CNN
+	1    2800 2400
+	0    -1   -1   0
+$EndComp
+$Comp
+L R R25
+U 1 1 5763B1A0
+P 2800 2650
+F 0 "R25" V 2880 2650 50  0000 C CNN
+F 1 "220" V 2800 2650 50  0000 C CNN
+F 2 "Resistors_SMD:R_0603_HandSoldering" V 2730 2650 50  0001 C CNN
+F 3 "" H 2800 2650 50  0000 C CNN
+	1    2800 2650
+	1    0    0    -1
+$EndComp
+Wire Wire Line
+	1650 2000 3150 2000
+Wire Wire Line
+	3150 2000 3150 2300
+Wire Wire Line
+	1650 2200 2800 2200
+Wire Wire Line
+	2800 2200 2800 2300
+Wire Wire Line
+	2800 2800 3300 2800
+Text GLabel 3300 2800 2    60   Input ~ 0
+LED_GND
+Connection ~ 3150 2800
+$Comp
+L Led_Small D15
+U 1 1 5763B807
+P 7550 1950
+F 0 "D15" H 7500 2075 50  0000 L CNN
+F 1 "MOSI" H 7550 1850 50  0000 L CNN
+F 2 "SMD_LED:LED_SMD_1.6x0.8mm" V 7550 1950 50  0001 C CNN
+F 3 "" V 7550 1950 50  0000 C CNN
+	1    7550 1950
+	0    -1   -1   0
+$EndComp
+$Comp
+L R R28
+U 1 1 5763B80D
+P 7550 2200
+F 0 "R28" V 7630 2200 50  0000 C CNN
+F 1 "220" V 7550 2200 50  0000 C CNN
+F 2 "Resistors_SMD:R_0603_HandSoldering" V 7480 2200 50  0001 C CNN
+F 3 "" H 7550 2200 50  0000 C CNN
+	1    7550 2200
+	1    0    0    -1
+$EndComp
+$Comp
+L Led_Small D14
+U 1 1 5763B813
+P 7200 1950
+F 0 "D14" H 7150 2075 50  0000 L CNN
+F 1 "MISO" H 7200 1850 50  0000 L CNN
+F 2 "SMD_LED:LED_SMD_1.6x0.8mm" V 7200 1950 50  0001 C CNN
+F 3 "" V 7200 1950 50  0000 C CNN
+	1    7200 1950
+	0    -1   -1   0
+$EndComp
+$Comp
+L R R27
+U 1 1 5763B819
+P 7200 2200
+F 0 "R27" V 7280 2200 50  0000 C CNN
+F 1 "220" V 7200 2200 50  0000 C CNN
+F 2 "Resistors_SMD:R_0603_HandSoldering" V 7130 2200 50  0001 C CNN
+F 3 "" H 7200 2200 50  0000 C CNN
+	1    7200 2200
+	1    0    0    -1
+$EndComp
+Wire Wire Line
+	7200 2350 7700 2350
+Text GLabel 7700 2350 2    60   Input ~ 0
+LED_GND
+Connection ~ 7550 2350
+Wire Wire Line
+	7550 1600 7550 1850
+Connection ~ 6600 1600
+Wire Wire Line
+	6250 2850 6850 2850
+Wire Wire Line
+	6850 2850 6850 1850
+Wire Wire Line
+	6850 1850 7200 1850
+Wire Wire Line
+	9200 3050 9200 2700
 $EndSCHEMATC
