File: kicad/Digital_Control.sch (KiCad schematic (older format))
At the start: 26 parts, among them IC1 ATMEGA328P-P, P10 ICSP, Q4 TSM2302CX, SW1 SW_PUSH, Y1 16MHz

Commit message: Updated board design with some footprint changes and improved audio layout
Parts:
- SW1: footprint Buttons_Switches_SMD:SW_SPST_B3S-1000 -> Buttons_Switches_SMD:SW_SPST_EVPBF
Changed lines of the file:
@@
 F 0 "SW1" H 8650 1510 50  0000 C CNN
 F 1 "SW_PUSH" H 8500 1320 50  0000 C CNN
-F 2 "Buttons_Switches_SMD:SW_SPST_B3S-1000" H 8500 1400 50  0001 C CNN
+F 2 "Buttons_Switches_SMD:SW_SPST_EVPBF" H 8500 1400 50  0001 C CNN
 F 3 "" H 8500 1400 50  0000 C CNN
 	1    8500 1400
